File: i5ether/i5ether.kicad_pcb (KiCad board)
At the start: 2 copper layers, 73 x 74 mm, 33 parts, among them J1 Conn_02x15_Odd_Even, J2 1-406541-1, J3 1-406541-1, T1 HX5008, T2 HX5008

Commit message: jlpcb fab files and small fixes to PCB
Other:
- net class Default removed
